File: VCA/VCA/VCA.kicad_sch (KiCad schematic)
At the start: 54 parts, among them J1 VCO1, J2 VCO2, J3 VCO3, J4 VCO4, J5 Q1, J6 Q2, J7 Q3, J8 Q2, U1 SSI2164, U2 LM324

Commit message: updated yo kengiz yawn guh bubby pirket
bubdaped yo dingdabing pep ring rong geeee renni
Parts:
- removed C10, C7, C8, C9: 100pF, symbol Device:C
- removed C? (x16): 560pF, symbol Device:C
- removed R10, R11, R12, R13: 30k, symbol Device:R
- added C? (x4): 100pF, symbol Device:C
- added R? (x4): 30k, symbol Device:R
Connections:
- net at U1.5 (I_OUT2), U2.6 (-): now also C?.2, R?.1
- net at J6.S, U2.7: now also C?.1, R?.2
- net at J5.S, U2.1: now also C?.1, R?.2
- net at U1.4 (I_OUT1), U2.2 (-): now also C?.2, R?.1
- net at J7.S, U2.8: now also C?.1, R?.2
- net at U1.12 (I_OUT3), U2.9 (-): now also C?.2, R?.1
- net at J8.S, U2.14: now also C?.1, R?.2
- net at U1.13 (I_OUT4), U2.13 (-): now also C?.2, R?.1
Other:
- moved on the sheet: C1, C2, C3, C4, C5, C6, J1, J2, J3, J4, J5, J6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

Commit message: eh
Parts:
- removed J1: VCO1, symbol Connector:AudioJack2_Ground
- removed J2: VCO2, symbol Connector:AudioJack2_Ground
- removed J3: VCO3, symbol Connector:AudioJack2_Ground
- removed J4: VCO4, symbol Connector:AudioJack2_Ground
- removed J5: Q1, symbol Connector:AudioJack2_Ground
- removed J6, J8: Q2, symbol Connector:AudioJack2_Ground
- removed J7: Q3, symbol Connector:AudioJack2_Ground
- removed J?: ADSR3, symbol Connector:AudioJack2_Ground
- removed J?: ADSR1, symbol Connector:AudioJack2_Ground
- removed J?: ADSR4, symbol Connector:AudioJack2_Ground
- removed J?: ADSR2, symbol Connector:AudioJack2_Ground
- added J1, J10, J11, J12, J2, J3, J4, J5, J6, J7, J8, J9: Conn_01x01_Pin, Connector_PinSocket_2.54mm:PinSocket_1x01_P2.54mm_Vertical, symbol Connector:Conn_01x01_Pin
- C1, C2, C3, C4, C5, C6: footprint (none) -> Capacitor_SMD:C_1206_3216Metric
- C10, C7, C8, C9: renamed from C?; footprint (none) -> Capacitor_SMD:C_1206_3216Metric
- J13: renamed from J?; footprint (none) -> Connector_PinSocket_2.54mm:PinSocket_2x05_P2.54mm_Vertical
- R1, R2, R3, R4, R5, R6, R7, R8, R9: footprint (none) -> Resistor_SMD:R_1206_3216Metric
- R10, R11, R12, R13: renamed from R?; footprint (none) -> Resistor_SMD:R_1206_3216Metric
- U2: footprint (none) -> Package_DIP:DIP-14_W7.62mm_Socket
Connections:
- net Out2: now reaches C8.1, R11.2, U2.7
- net Out2: now also J6.1 (Pin_1)
- net Out3: now reaches C9.1, R12.2, U2.8
- net Out3: now also J7.1 (Pin_1)
- net VCO1: now reaches R1.1
- net VCO1: now also J1.1 (Pin_1)
- net VCO3: now reaches R5.1
- net VCO3: now also J3.1 (Pin_1)
- net ADSR3: now reaches U1.11 (VC3)
- net ADSR3: now also J10.1 (Pin_1)
- net Out1: now reaches C7.1, R10.2, U2.1
- net Out1: now also J5.1 (Pin_1)
- net VCO4: now reaches R7.1
- net VCO4: now also J4.1 (Pin_1)
- net ADSR1: now reaches U1.3 (VC1)
- net ADSR1: now also J12.1 (Pin_1)
- net Out4: now reaches C10.1, R13.2, U2.14
- net Out4: now also J8.1 (Pin_1)
- net ADSR4: now reaches U1.14 (VC4)
- net ADSR4: now also J9.1 (Pin_1)
- net VCO2: now reaches R3.1
- net VCO2: now also J2.1 (Pin_1)
- net ADSR2: now reaches U1.6 (VC2)
- net ADSR2: now also J11.1 (Pin_1)
