File: Low Noise Power Supply/Power supply -SCH & PCB/Power supply.kicad_pcb (KiCad board)
At the start: 2 copper layers, 91.4 x 35.6 mm, 27 parts, among them J4 12VA, J5 GND, U1 LM7812_TO220, U2 LM7912_TO220

Commit message: power
Parts:
- added REF**: BarrelJack_CUI_PJ-063AH_Horizontal, Connector_BarrelJack:BarrelJack_CUI_PJ-063AH_Horizontal, F.Cu at (88.9, 95.9)
- moved D4 15.7 mm to (83.2, 112.4), turned to 0 degrees
- moved J4 8.52 mm to (78.7, 87.6), turned to 180 degrees
- moved J5 8.03 mm to (78.7, 104.1)
- moved REF** 7.62 mm to (78.7, 111.8)
- moved REF** 7.62 mm to (78.7, 81.3)
- moved D2 3.70 mm to (93.3, 80.6), turned to 180 degrees
Routing:
- net +12VA: track 11.2 -> 41.3 mm
- net Net-(D4-A): track 75.8 -> 75.2 mm
Other:
- board size 91.4 x 35.6 mm -> 99.1 x 35.6 mm
- board text added: "<-- 12v AC <-- Bypass"
- board text added: "<-- GND <-- Bypass"

Commit message: minor power supply changes
Other:
- board text added: "Certain Synthesizers 12V AC to +/-12V DC Low Noise 6/9/2023 Rev 2.0"
- board text removed: "Certain Synthesizers 12V AC to +/-12V DC Low Noise 6/8/2023"
