File: VCO Remake/as3340_no_mux/as3340_no_mux.kicad_pcb (KiCad board)
At the start: 4 copper layers, 20.3 x 118.1 mm, 61 parts, among them J1 Sync INput, J11 Conn_02x05_Odd_Even, J12 TRI OUt, J13 SIN OUT, J14 SAW OUt, J15 SQR OUT, J2 CV1, J4 LinearFmINput, J5 PWM INput, U1 LM13700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

Commit message: eh
Parts:
- added J10: Conn_01x01_Male, Connector_PinHeader_2.54mm:PinHeader_1x01_P2.54mm_Vertical, F.Cu at (103.8, 62.7)
- added J16: Conn_01x01_Male, Connector_PinHeader_2.54mm:PinHeader_1x01_P2.54mm_Vertical, F.Cu at (103.8, 67.4)
- added J17: Conn_01x01_Male, Connector_PinHeader_2.54mm:PinHeader_1x01_P2.54mm_Vertical, F.Cu at (103.8, 72.0)
- added J18: Conn_01x01_Male, Connector_PinHeader_2.54mm:PinHeader_1x01_P2.54mm_Vertical, F.Cu at (103.8, 76.7)
- added J19: Conn_01x01_Male, Connector_PinHeader_2.54mm:PinHeader_1x01_P2.54mm_Vertical, F.Cu at (103.8, 81.3)
- added J20: Conn_01x01_Male, Connector_PinHeader_2.54mm:PinHeader_1x01_P2.54mm_Vertical, F.Cu at (108.5, 62.7)
- added J21: Conn_01x01_Male, Connector_PinHeader_2.54mm:PinHeader_1x01_P2.54mm_Vertical, F.Cu at (108.5, 67.4)
- added J22: Conn_01x06_Female, Connector_PinHeader_2.54mm:PinHeader_1x06_P2.54mm_Vertical, F.Cu at (117.8, 62.7)
- added J23: Conn_01x06_Male, Connector_PinHeader_2.54mm:PinHeader_1x06_P2.54mm_Vertical, F.Cu at (122.4, 62.7)
- added J24: Conn_01x01_Male, Connector_PinHeader_2.54mm:PinHeader_1x01_P2.54mm_Vertical, F.Cu at (108.5, 72.0)
- added J25: Conn_01x01_Male, Connector_PinHeader_2.54mm:PinHeader_1x01_P2.54mm_Vertical, F.Cu at (108.5, 76.7)
- added J26: Conn_01x01_Male, Connector_PinHeader_2.54mm:PinHeader_1x01_P2.54mm_Vertical, F.Cu at (108.5, 81.3)
- added J27: Conn_01x01_Male, Connector_PinHeader_2.54mm:PinHeader_1x01_P2.54mm_Vertical, F.Cu at (113.1, 62.7)
- added J28: Conn_01x01_Male, Connector_PinHeader_2.54mm:PinHeader_1x01_P2.54mm_Vertical, F.Cu at (113.1, 67.4)
- added J29: Conn_01x01_Male, Connector_PinHeader_2.54mm:PinHeader_1x01_P2.54mm_Vertical, F.Cu at (113.1, 72.0)
- added J3: Conn_01x01_Male, Connector_PinHeader_2.54mm:PinHeader_1x01_P2.54mm_Vertical, F.Cu at (99.2, 62.7)
- added J30: Conn_01x01_Male, Connector_PinHeader_2.54mm:PinHeader_1x01_P2.54mm_Vertical, F.Cu at (113.1, 76.7)
- added J6: Conn_01x01_Male, Connector_PinHeader_2.54mm:PinHeader_1x01_P2.54mm_Vertical, F.Cu at (99.2, 67.4)
- added J7: Conn_01x01_Male, Connector_PinHeader_2.54mm:PinHeader_1x01_P2.54mm_Vertical, F.Cu at (99.2, 72.0)
- added J8: Conn_01x01_Male, Connector_PinHeader_2.54mm:PinHeader_1x01_P2.54mm_Vertical, F.Cu at (99.2, 76.7)
- added J9: Conn_01x01_Male, Connector_PinHeader_2.54mm:PinHeader_1x01_P2.54mm_Vertical, F.Cu at (99.2, 81.3)
- added SW1: SW_SPDT, Potentiometer_THT:Potentiometer_ACP_CA6-H2,5_Horizontal, F.Cu at (117.1, 79.4)
Other:
- copper layers 4 -> 2

Commit message: Very Epic 2 layer VCO
Parts:
- removed J10, J16, J17, J18, J19, J20, J21, J24, J25, J26, J27, J28, J29, J3, J30, J6, J7, J8, J9: Conn_01x01_Male, Connector_PinHeader_2.54mm:PinHeader_1x01_P2.54mm_Vertical
- removed J22: Conn_01x06_Female, Connector_PinHeader_2.54mm:PinHeader_1x06_P2.54mm_Vertical
- removed J23: Conn_01x06_Male, Connector_PinHeader_2.54mm:PinHeader_1x06_P2.54mm_Vertical
- added R5: 20K, Resistor_SMD:R_1206_3216Metric, B.Cu at (196.9, 51.5)
- added R7: 470, Resistor_SMD:R_1206_3216Metric, B.Cu at (189.0, 88.7)
- added R9: 47k, Resistor_SMD:R_1206_3216Metric, B.Cu at (186.4, 134.9)
- added THONKY_COURSE_CV1: 100k Pot, Potentiometer_THT:Potentiometer_Alps_RK09K_Single_Vertical, F.Cu at (185.5, 43.8)
- added THONKY_FINE_CV1: 100k Pot, Potentiometer_THT:Potentiometer_Alps_RK09K_Single_Vertical, F.Cu at (185.5, 58.4)
- added THONKY_PWM1: 100k Pot, Potentiometer_THT:Potentiometer_Alps_RK09K_Single_Vertical, F.Cu at (185.5, 73.0)
- NOT+THINKY_CV1: renamed from RV7; footprint Potentiometer_THT:Potentiometer_Alps_RK09K_Single_Vertical -> Potentiometer_THT:Potentiometer_ACP_CA6-H2,5_Horizontal; moved to B.Cu
- NOT_THINKY_TEMKO1: renamed from RV9; footprint Potentiometer_THT:Potentiometer_Alps_RK09K_Single_Vertical -> Potentiometer_THT:Potentiometer_ACP_CA6-H2,5_Horizontal; moved to B.Cu
- NOT_THONKY_HF_TRACK1: renamed from RV5; value 20k Pot -> 10k Pot; footprint Potentiometer_THT:Potentiometer_Alps_RK09K_Single_Vertical -> Potentiometer_THT:Potentiometer_ACP_CA6-H2,5_Horizontal; moved to B.Cu
- SW1: moved to B.Cu
- moved R19 103.1 mm to (179.2, 139.7)
- moved R17 99.2 mm to (192.9, 132.2), turned to 0 degrees
- moved R39 87.6 mm to (182.8, 133.7)
- moved SW1 80.6 mm to (197.0, 68.7), turned to 180 degrees
- moved R26 75.1 mm to (197.0, 136.9), turned to 90 degrees
- moved R11 71.4 mm to (188.8, 103.0)
- moved C7 70.1 mm to (183.1, 103.0)
- moved R40 62.9 mm to (189.4, 132.2)
- moved R67 61.8 mm to (196.8, 132.2), turned to 90 degrees
- moved R4 59.7 mm to (196.9, 141.6)
- moved R66 59.2 mm to (196.9, 109.3), turned to 90 degrees
- moved R12 56.5 mm to (188.8, 100.6), turned to 0 degrees
- moved C9 55.1 mm to (188.6, 92.5)
- moved R1 55.0 mm to (196.9, 94.1), turned to 90 degrees
- moved C3 53.7 mm to (197.0, 104.5)
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- renumbered SineLevelTrim1 to NOT_THINK_SineLevelTrim1, SineShapeTrim1 to NOT_THONKY_SineShapeTrim1, SineBiasTrim1 to NOT_THOONKY_SineBiasTrim1, C11 to PolyStirene!C11
Connections:
- C3 pad 1: Net-(J10-Pin_1) -> Net-(SW1-C)
- C7 pad 1: Net-(J9-Pin_1) -> Net-(SW1-A)
- J1 pad T: Net-(J25-Pin_1) -> Net-(SW1-B)
- R24 pad 1: Net-(U2-VFCI) -> Net-(J2-PadR)
- R24 pad 2: Net-(J2-PadR) -> Net-(U2-VFCI)
- R58 pad 1: Net-(J23-Pin_4) -> Net-(U2-VP)
- SW1 pad 1: Net-(J7-Pin_1) -> Net-(SW1-A)
- SW1 pad 2: Net-(J24-Pin_1) -> Net-(SW1-B)
- SW1 pad 3: Net-(J8-Pin_1) -> Net-(SW1-C)
- U2 pad 10: Net-(J22-Pin_1) -> Net-(U2-VTO)
- U2 pad 4: Net-(J22-Pin_4) -> Net-(U2-VP)
- U2 pad 8: Net-(J22-Pin_5) -> Net-(U2-VSO)
- U4 pad 12: Net-(J23-Pin_5) -> Net-(U2-VSO)
- U4 pad 5: Net-(J23-Pin_1) -> Net-(U2-VTO)
Routing:
- net GND: track 0.00 -> 280.8 mm, vias 0 -> 3
- net +15V: track 0.00 -> 164.2 mm, vias 0 -> 2
- net -15V: track 0.00 -> 147.1 mm, vias 0 -> 1
- net Net-(NOT+THINKY_CV1-Pad1): track 0.00 -> 124.1 mm, vias 0 -> 1
- net Net-(U2-VFCI): track 0.00 -> 105.2 mm, vias 0 -> 1
- net Net-(NOT_THONKY_HF_TRACK1-Pad2): track 0.00 -> 101.3 mm, vias 0 -> 1
- net Net-(NOT_THINKY_TEMKO1-Pad1): track 0.00 -> 90.5 mm, vias 0 -> 1
- net Net-(D1-A): track 0.00 -> 89.4 mm, vias 0 -> 4
- net Net-(U2-VEE): track 0.00 -> 87.4 mm, vias 0 -> 2
- net Net-(R19-Pad1): track 0.00 -> 84.6 mm, vias 0 -> 1
- net Net-(U2-VHFT): track 0.00 -> 78.6 mm, vias 0 -> 1
- net Net-(NOT_THONKY_SineShapeTrim1-Pad1): track 0.00 -> 73.8 mm, vias 0 -> 2
- net Net-(U2-VSO): track 0.00 -> 72.6 mm, vias 0 -> 1
- net Net-(U2-VLFI): track 0.00 -> 68.0 mm, vias 0 -> 2
- net Net-(J5-PadR): track 0.00 -> 65.5 mm
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- added copper zone on B.Cu, net GND
- added copper zone on F.Cu, net GND

Commit message: How????
Parts:
- PolyStirene!C11: footprint Capacitor_SMD:C_1206_3216Metric -> Capacitor_THT:C_Radial_D5.0mm_H5.0mm_P2.00mm
- moved R46 2.91 mm to (191.0, 134.5), turned to 0 degrees
- moved R17 2.28 mm to (194.6, 133.7), turned to 90 degrees
- moved PolyStirene!C11 1.67 mm to (189.6, 139.7)
- moved R40 1.63 mm to (191.0, 132.1), turned to 0 degrees
- moved J11 0.12 mm to (193.0, 146.7)
Routing:
- net +15V: track 164.2 -> 204.4 mm, vias 2 -> 1
- net -15V: track 147.1 -> 173.7 mm
- net GND: track 280.8 -> 254.3 mm, vias 3 -> 2
- net Net-(U2-VFCI): track 105.2 -> 81.7 mm, vias 1 -> 2
- net Net-(U2-VLFI): track 68.0 -> 48.2 mm, vias 2 -> 4
- net Net-(U2-VEE): track 87.4 -> 103.5 mm, vias 2 -> 1
- net Net-(NOT_THONKY_HF_TRACK1-Pad2): track 101.3 -> 117.1 mm, vias 1 -> 2
- net Net-(SW1-A): track 54.5 -> 40.5 mm
- net Net-(NOT_THINKY_TEMKO1-Pad1): track 90.5 -> 102.3 mm, vias 1 -> 6
- net Net-(U2-VSO): track 72.6 -> 81.7 mm, vias 1 -> 3
- net Net-(U2-VPWM): track 49.2 -> 57.5 mm, vias 2 -> 0
- net Net-(J5-PadR): track 65.5 -> 73.0 mm
- net Net-(U4B--): track 11.6 -> 17.3 mm
- net Net-(SW1-B): track 64.7 -> 59.0 mm
- net Net-(R3-Pad1): track 20.7 -> 15.3 mm, vias 0 -> 2
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