File: VCO Remake/as3340_no_mux/as3340_no_mux.kicad_pcb (KiCad board)
At the start: 2 copper layers, 49.5 x 128.5 mm, 87 parts, among them J1 Sync INput, J11 Conn_02x05_Odd_Even, J12 TRI OUt, J13 SIN OUT, J14 SAW OUt, J15 SQR OUT, J2 CV1, J4 LinearFmINput, J5 PWM INput, SW1 SW_SPDT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

Commit message: HUGE VCO UPDATE FOR AUTOMATION
Parts:
- removed G*** (x7): LOGO, LOGO
- removed SLOTMAN, Slot1, Slot10, Slot2, Slot3, Slot33, Slot4, Slot87, Slot9: CV1, AudioJacks:Jack_3.5mm_QingPu_WQP-PJ398SM_Vertical
- removed the THONKY_COURSE_CV1 at (214.7, 43.6)
- removed the THONKY_FINE_CV1 at (214.7, 58.2)
- removed the THONKY_PWM1 at (214.7, 72.9)
Other:
- board size 49.5 x 128.5 mm -> 20.3 x 118.1 mm
- board text removed: "100k"
- board text removed: "20k"
- board text removed: "470k"
- board text removed: "Certain Synths VCO"
- board text removed: "Course Tune"
- board text removed: "Fine Tune"
- board text removed: "Pulse Width"
