File: VCO4_JLC_AUTOMATION/as3340_no_mux/as3340_no_mux.kicad_sch (KiCad schematic)
At the start: 66 parts, among them J1 Sync INput, J11 Conn_02x05_Odd_Even, J12 TRI OUt, J13 SIN OUT, J14 SAW OUt, J15 SQR OUT, J2 CV1, J4 LinearFmINput, J5 PWM INput, SW1 SW_SPDT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

Commit message: L
Parts:
- R12: footprint Resistor_SMD:R_1206_3216Metric -> Resistor_SMD:R_0805_2012Metric
Changed lines of the file:
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@@
       (effects (font (size 1.27 1.27)))
     )
-    (property "Footprint" "Resistor_SMD:R_1206_3216Metric" (at 165.1 112.522 90)
+    (property "Footprint" "Resistor_SMD:R_0805_2012Metric" (at 165.1 112.522 90)
       (effects (font (size 1.27 1.27)) hide)
     )
