File: VCO4_JLC_AUTOMATION/as3340_no_mux/as3340_no_mux.kicad_pcb (KiCad board)
At the start: 2 copper layers, 20.3 x 118.1 mm, 66 parts, among them J1 Sync INput, J11 Conn_02x05_Odd_Even, J12 TRI OUt, J13 SIN OUT, J14 SAW OUt, J15 SQR OUT, J2 CV1, J4 LinearFmINput, J5 PWM INput, SW1 SW_SPDT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

Commit message: L
Parts:
- R12: footprint Resistor_SMD:R_1206_3216Metric -> Resistor_SMD:R_0805_2012Metric
Routing:
- net Net-(U2-VLFI): track 51.4 -> 51.9 mm
Changed lines of the file:
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@@
     )
   )
-  (footprint "Resistor_SMD:R_1206_3216Metric" (layer "B.Cu")
+  (footprint "Resistor_SMD:R_0805_2012Metric" (layer "B.Cu")
     (at 188.7728 100.584)
-    (descr "Resistor SMD 1206 (3216 Metric), square (rectangular) end terminal, IPC_7351 nominal, (Body size source: IPC-SM-782 page 72, https://www.pcb-3d.com/wordpress/wp-content/uploads/ipc-sm-782a_amendment_1_and_2.pdf), generated with kicad-footprint-generator")
+    (descr "Resistor SMD 0805 (2012 Metric), square (rectangular) end terminal, IPC_7351 nominal, (Body size source: IPC-SM-782 page 72, https://www.pcb-3d.com/wordpress/wp-content/uploads/ipc-sm-782a_amendment_1_and_2.pdf), generated with kicad-footprint-generator")
     (tags "resistor")
     (property "Sheetfile" "as3340_no_mux.kicad_sch")
@@
     (property "ki_keywords" "R res resistor")
     (attr smd)
-    (fp_text reference "R12" (at 0 1.82) (layer "B.SilkS")
-        (effects (font (size 1 1) (thickness 0.15)) (justify mirror))
-    )
-    (fp_text value "470" (at 0 -1.82) (layer "B.Fab")
-        (effects (font (size 1 1) (thickness 0.15)) (justify mirror))
-    )
-    (fp_text user "${REFERENCE}" (at 0 0) (layer "B.Fab")
-        (effects (font (size 0.8 0.8) (thickness 0.12)) (justify mirror))
-    )
-    (fp_line (start -0.727064 -0.91) (end 0.727064 -0.91)
-      (stroke (width 0.12) (type solid)) (layer "B.SilkS"))
-    (fp_line (start -0.727064 0.91) (end 0.727064 0.91)
-      (stroke (width 0.12) (type solid)) (layer "B.SilkS"))
-    (fp_line (start -2.28 -1.12) (end -2.28 1.12)
-      (stroke (width 0.05) (type solid)) (layer "B.CrtYd"))
-    (fp_line (start -2.28 1.12) (end 2.28 1.12)
-      (stroke (width 0.05) (type solid)) (layer "B.CrtYd"))
-    (fp_line (start 2.28 -1.12) (end -2.28 -1.12)
-      (stroke (width 0.05) (type solid)) (layer "B.CrtYd"))
-    (fp_line (start 2.28 1.12) (end 2.28 -1.12)
-      (stroke (width 0.05) (type solid)) (layer "B.CrtYd"))
-    (fp_line (start -1.6 -0.8) (end -1.6 0.8)
-      (stroke (width 0.1) (type solid)) (layer "B.Fab"))
-    (fp_line (start -1.6 0.8) (end 1.6 0.8)
-      (stroke (width 0.1) (type solid)) (layer "B.Fab"))
-    (fp_line (start 1.6 -0.8) (end -1.6 -0.8)
-      (stroke (width 0.1) (type solid)) (layer "B.Fab"))
-    (fp_line (start 1.6 0.8) (end 1.6 -0.8)
-      (stroke (width 0.1) (type solid)) (layer "B.Fab"))
-    (pad "1" smd roundrect (at -1.4625 0) (size 1.125 1.75) (layers "B.Cu" "B.Paste" "B.Mask") (roundrect_rratio 0.2222222222)
+    (fp_text reference "R12" (at 0 1.65 180) (layer "B.SilkS")
+        (effects (font (size 1 1) (thickness 0.15)) (justify mirror))
+    )
+    (fp_text value "470" (at 0 -1.65 180) (layer "B.Fab")
+        (effects (font (size 1 1) (thickness 0.15)) (justify mirror))
+    )
+    (fp_text user "${REFERENCE}" (at 0 0 180) (layer "B.Fab")
+        (effects (font (size 0.5 0.5) (thickness 0.08)) (justify mirror))
+    )
+    (fp_line (start -0.227064 -0.735) (end 0.227064 -0.735)
+      (stroke (width 0.12) (type solid)) (layer "B.SilkS"))
+    (fp_line (start -0.227064 0.735) (end 0.227064 0.735)
+      (stroke (width 0.12) (type solid)) (layer "B.SilkS"))
+    (fp_line (start -1.68 -0.95) (end -1.68 0.95)
+      (stroke (width 0.05) (type solid)) (layer "B.CrtYd"))
+    (fp_line (start -1.68 0.95) (end 1.68 0.95)
+      (stroke (width 0.05) (type solid)) (layer "B.CrtYd"))
+    (fp_line (start 1.68 -0.95) (end -1.68 -0.95)
+      (stroke (width 0.05) (type solid)) (layer "B.CrtYd"))
+    (fp_line (start 1.68 0.95) (end 1.68 -0.95)
+      (stroke (width 0.05) (type solid)) (layer "B.CrtYd"))
+    (fp_line (start -1 -0.625) (end -1 0.625)
+      (stroke (width 0.1) (type solid)) (layer "B.Fab"))
+    (fp_line (start -1 0.625) (end 1 0.625)
+      (stroke (width 0.1) (type solid)) (layer "B.Fab"))
+    (fp_line (start 1 -0.625) (end -1 -0.625)
+      (stroke (width 0.1) (type solid)) (layer "B.Fab"))
+    (fp_line (start 1 0.625) (end 1 -0.625)
+      (stroke (width 0.1) (type solid)) (layer "B.Fab"))
+    (pad "1" smd roundrect (at -0.9125 0) (size 1.025 1.4) (layers "B.Cu" "B.Paste" "B.Mask") (roundrect_rratio 0.243902439)
       (net 22 "Net-(U2-VLFI)") (pintype "passive"))
-    (pad "2" smd roundrect (at 1.4625 0) (size 1.125 1.75) (layers "B.Cu" "B.Paste" "B.Mask") (roundrect_rratio 0.2222222222)
+    (pad "2" smd roundrect (at 0.9125 0) (size 1.025 1.4) (layers "B.Cu" "B.Paste" "B.Mask") (roundrect_rratio 0.243902439)
       (net 4 "Net-(C2-Pad2)") (pintype "passive"))
-    (model "${KICAD6_3DMODEL_DIR}/Resistor_SMD.3dshapes/R_1206_3216Metric.wrl"
+    (model "${KICAD6_3DMODEL_DIR}/Resistor_SMD.3dshapes/R_0805_2012Metric.wrl"
       (offset (xyz 0 0 0))
       (scale (xyz 1 1 1))
@@
   (segment (start 191.4752 128.5435) (end 191.4752 130.5121) (width 0.2) (layer "B.Cu") (net 3))
   (segment (start 191.9205 134.5846) (end 190.7186 135.7865) (width 0.2) (layer "B.Cu") (net 3))
+  (segment (start 189.28815 99.63685) (end 189.28815 100.18685) (width 0.2) (layer "B.Cu") (net 4))
   (segment (start 188.4455 97.6259) (end 185.1742 94.3546) (width 0.2) (layer "B.Cu") (net 4))
+  (segment (start 189.28815 99.63685) (end 188.4455 98.7942) (width 0.2) (layer "B.Cu") (net 4))
   (segment (start 185.1742 94.3546) (end 180.7672 94.3546) (width 0.2) (layer "B.Cu") (net 4))
   (segment (start 180.7672 94.3546) (end 179.324 92.9114) (width 0.2) (layer "B.Cu") (net 4))
-  (segment (start 190.2353 100.584) (end 188.4455 98.7942) (width 0.2) (layer "B.Cu") (net 4))
   (segment (start 188.4455 98.7942) (end 188.4455 97.6259) (width 0.2) (layer "B.Cu") (net 4))
+  (segment (start 189.28815 100.18685) (end 189.6853 100.584) (width 0.2) (layer "B.Cu") (net 4))
   (segment (start 190.7899 114.0576) (end 191.9721 112.8754) (width 0.2) (layer "B.Cu") (net 5))
   (segment (start 188.7421 114.0576) (end 190.7899 114.0576) (width 0.2) (layer "B.Cu") (net 5))
@@
   (segment (start 187.492 102.8915) (end 188.4688 102.8915) (width 0.2) (layer "B.Cu") (net 22))
   (segment (start 187.3611 103.0224) (end 187.492 102.8915) (width 0.2) (layer "B.Cu") (net 22))
+  (segment (start 187.3103 100.584) (end 187.8603 100.584) (width 0.2) (layer "B.Cu") (net 22))
   (segment (start 191.1029 85.3551) (end 189.5143 85.3551) (width 0.2) (layer "B.Cu") (net 22))
   (segment (start 185.5462 112.9536) (end 187.3785 111.1213) (width 0.2) (layer "F.Cu") (net 23))

Commit message: e
Changed lines of the file:
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@@
     (fp_rect (start -1.651 -3.431) (end 11.049 3.429)
       (stroke (width 0.1) (type default)) (fill none) (layer "F.SilkS"))
-    (pad "1" thru_hole circle (at 0 0) (size 1.7 1.7) (drill 0.9) (layers "*.Cu" "*.Mask")
+    (pad "1" thru_hole circle (at 0 0) (size 1.7 1.7) (drill oval 0.9 1.25) (layers "*.Cu" "*.Mask")
       (net 24 "Net-(SW1-A)") (pinfunction "A") (pintype "passive"))
-    (pad "2" thru_hole circle (at 4.7 0) (size 1.7 1.7) (drill 0.9) (layers "*.Cu" "*.Mask")
+    (pad "2" thru_hole circle (at 4.7 0) (size 1.7 1.7) (drill oval 0.9 1.25) (layers "*.Cu" "*.Mask")
       (net 25 "Net-(SW1-B)") (pinfunction "B") (pintype "passive"))
-    (pad "3" thru_hole circle (at 9.4 0) (size 1.7 1.7) (drill 0.9) (layers "*.Cu" "*.Mask")
+    (pad "3" thru_hole circle (at 9.4 0) (size 1.7 1.7) (drill oval 0.9 1.25) (layers "*.Cu" "*.Mask")
       (net 20 "Net-(SW1-C)") (pinfunction "C") (pintype "passive"))
     (model "${KICAD6_3DMODEL_DIR}/Button_Switch_THT.3dshapes/SW_E-Switch_EG1224_SPDT_Angled.wrl"
