File: VCO Remake/as3340_Front_panel/VCOFRONTPANEL/VCOFRONTPANEL.kicad_pcb (KiCad board)
At the start: 2 copper layers, 20.3 x 128.5 mm, 19 parts

Commit message: e
Parts:
- moved G*** 1.02 mm to (154.2, 108.0)
